File: Electronics/Ahoge/_restore_backup_2026-07-16T16-28-27-267/Ahoge.kicad_sch (KiCad schematic)
At the start: 7 parts, among them M1 Motor_DC, M2 Motor_DC, SW1 SW_Push_SPDT, SW2 SW_Push_SPDT, U1 L9110, U2 L9110

Commit message: mis
Parts:
- removed M2: Motor_DC, symbol k:Motor_DC
- removed U1, U2: L9110, symbol import:L9110
Connections:
- net at M1.1 (+): now also RZ1.3 (GP2)
- net at M1.2 (-): now also RZ1.4 (GP3)
Other:
- moved on the sheet: M1
